File: hardware/girth/PCB/kicad/AVO_GIRTH_PCB.kicad_sch (KiCad schematic)
At the start: 93 parts, among them J1 USB-C 16P, J2 BATERÍA 1S, Q1 AO3401A, Q2 AO3401A, Q3 AO3401A, SW1 REED (1), SW2 REED (2), U1 BQ51013BRHLR, U2 BQ24072RGTR, U3 RT9080-33GJ5, U4 ESP32-C6-MINI-1U-N4, U5 BNO085, U6 USBLC6-2SC6, Y1 32,768 kHz 12,5 pF

Commit message: PCB cincha REV A: corte de batería con relé biestable G6KU + ruteado con Freerouting en CI
- K1 G6KU-2F-Y DC3: se cierra con el pulso del reed o de los 5 V de carga, el ESP32 lo abre (GPIO23).
- Arranque suave con PMOS tras el relé; reed leído por Q16 (GPIO6).
- La placa de colocación lleva las vías a planos; Freerouting rutea el resto en el CI.

Co-Authored-By: Claude Opus 5.5 <noreply@anthropic.com>
Claude-Session: https://claude.ai/code/session_01CHDvF8BfHwPLkrFs9S3ECm
Parts:
- added C40, C41: 220u 6V3 polímero, AVO:CP_EIA-3528-21_Kemet-B, symbol AVO:C_avo
- added C43: 100n, AVO:C_0402_1005Metric, symbol AVO:C_avo
- added D10: BAT54C, AVO:SOT-23, symbol AVO:BAT54C_D
- added K1: G6KU-2F-Y DC3, AVO:Relay_DPDT_Omron_G6K-2F-Y, symbol AVO:G6KU-2F-Y_K
- added Q10, Q14: AO3401A, AVO:SOT-23, symbol AVO:AO3401A_Q
- added Q11, Q13: AO3400A, AVO:SOT-23, symbol AVO:AO3400A_Q
- added Q12, Q15, Q16: 2N7002, AVO:SOT-23, symbol AVO:2N7002_Q
- added R40, R41: 0R, AVO:R_0805_2012Metric, symbol AVO:R_avo
- added R44, R45: 10k, AVO:R_0402_1005Metric, symbol AVO:R_avo
- added R46, R47, R48, R49: 100k, AVO:R_0402_1005Metric, symbol AVO:R_avo
- added R50, R51: 1M, AVO:R_0402_1005Metric, symbol AVO:R_avo
- R31: value 1M -> 100k; LCSC C26083 -> C25741
Connections:
- net GND: now also Q11.2 (S), Q12.2 (S), Q13.2 (S), Q15.2 (S), Q16.2 (S), R44.2, R46.2, R48.2, R50.2, R51.2; no longer SW2.1
- net REED: now also Q16.3 (D); no longer SW1.1
- net VBAT: now also Q10.2 (S), Q14.3 (D), R47.2; no longer J2.1 (+)
- net VIN5: now also D10.2 (A2)
- net RLY_OFF: now reaches U4.29 (IO23 RELÉ OFF)
- net RLY_OFF: now also Q12.1 (G), Q13.1 (G), Q15.1 (G), R48.1
- new net BAT_RAW: J2.1 (+), K1.3 (COM1), K1.6 (COM2), SW2.1
- new net BAT_SW: C43.1, Q10.3 (D), R40.2, R41.2
- new net K_A: C40.2, C41.2, K1.1 (BOBINA A), Q13.3 (D)
- new net K_B: K1.8 (BOBINA B), Q11.3 (D), Q14.2 (S)
- new net REED_G: Q16.1 (G), R49.2, R50.1
- new net REED_HI: D10.1 (A1), R49.1, SW1.1
- new net RLY_GB: Q11.1 (G), Q12.3 (D), R45.2, R46.1
- new net RLY_NC: K1.2 (NC1), K1.7 (NC2), R41.1
- new net RLY_NO: K1.4 (NA1), K1.5 (NA2), R40.1
- new net RLY_P: C40.1, C41.1, D10.3 (K), R44.1, R45.1
- new net RLY_PG: Q14.1 (G), Q15.3 (D), R47.1
- new net SS_G: C43.2, Q10.1 (G), R51.1
- no-connect marks 22 -> 21
Other:
- note added: "CORTE DE BATERÍA: relé biestable G6KU"
- moved on the sheet: C15, C16, C17, C18, C19, C2, C20, C21, C22, C23, C24, C25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

Commit message: PCB cincha: relé también se cierra desde el ESP32 (GPIO14), puerta de fabricación en CI, reparación de ruteado
- Relé: camino SET por firmware (Q17/Q18/D11/R52–R55): con la base puesta el ESP32 vive del camino de potencia del
  cargador y puede volver a cerrar el relé → el sistema nunca queda bloqueado apagado.
- GND de las QFN unidos a su pad térmico por pistas cortas (sin vías que tapen la salida de los pines vecinos).
- Referencias en la capa Fab; huellas enlazadas a los símbolos (DRC con paridad de esquema).
- CI: puerta bloqueante (0 errores DRC, 0 incompletas, 0 paridad, ERC limpio); ficheros FINAL solo si pasa; rojo si no.
- fuente/repair.py: completa las conexiones que deja Freerouting y genera la placa ruteada que usa el CI.

Co-Authored-By: Claude Opus 5.5 <noreply@anthropic.com>
Claude-Session: https://claude.ai/code/session_01CHDvF8BfHwPLkrFs9S3ECm
Parts:
- added D11: BAT54C, AVO:SOT-23, symbol AVO:BAT54C_D
- added Q17: AO3401A, AVO:SOT-23, symbol AVO:AO3401A_Q
- added Q18: 2N7002, AVO:SOT-23, symbol AVO:2N7002_Q
- added R52: 10R, AVO:R_0805_2012Metric, symbol AVO:R_avo
- added R53, R54: 100k, AVO:R_0402_1005Metric, symbol AVO:R_avo
- added R55: 1k, AVO:R_0402_1005Metric, symbol AVO:R_avo
Connections:
- net GND: now also Q18.2 (S), R54.2
- net K_A: now also R52.2
- net RLY_GB: now also D11.3 (K)
- net VSYS: now also Q17.3 (D), R53.2
- net RLY_ON: now reaches U4.19 (IO14 RELÉ ON)
- net RLY_ON: now also Q18.1 (G), R54.1, R55.1
- new net K_A_SET: Q17.2 (S), R52.1
- new net RLY_ON_D: D11.1 (A1), R55.2
- new net RLY_SG: Q17.1 (G), Q18.3 (D), R53.1
Other:
- moved on the sheet: K1, Q10, Q11, Q12, Q13, Q14, Q15

Commit message: PCB cincha: In2 como capa de ruteado (+3V3 rellena después), pines abiertos con su nombre de red, esquema sin solapes, condensadores Qi separados de los pines, reparación con rip-up
Co-Authored-By: Claude Opus 5.5 <noreply@anthropic.com>
Claude-Session: https://claude.ai/code/session_01CHDvF8BfHwPLkrFs9S3ECm
Connections:
- net +3V3: now also Q3.2 (S); no longer Q3.3 (D)
- net AD_SRC: now also Q1.3 (D), Q2.3 (D); no longer Q1.2 (S), Q2.2 (S)
- net BAT_SW: now also Q10.2 (S); no longer Q10.3 (D)
- net IMU_VDD: now also Q3.3 (D); no longer Q3.2 (S)
- net K_A_SET: now also Q17.3 (D); no longer Q17.2 (S)
- net K_B: now also Q14.3 (D); no longer Q14.2 (S)
- net VBAT: now also Q10.3 (D), Q14.2 (S); no longer Q10.2 (S), Q14.3 (D)
- net VBUS: now also Q1.2 (S); no longer Q1.3 (D)
- net VIN5: now also Q2.2 (S); no longer Q2.3 (D)
- net VSYS: now also Q17.2 (S); no longer Q17.3 (D)
Other:
- note added: "Generado por fuente/avo_girth_pcb.py (mismo origen de datos que la placa). Las conexiones son etiquetas globales: dos pines con la misma etiqueta están unidos."
- note removed: "Generado por fuente/avo_girth_pcb.py (mismo origen de datos que la placa). Todas las conexiones son etiquetas de red: dos pines con la misma etiqueta están unidos."
- moved on the sheet: C1, C10, C11, C12, C13, C14, C15, C16, C17, C18, C19, C2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

Commit message: PCB cincha: entorno del BQ51013B reordenado (salida limpia de pines), símbolos por disposición de pines
Co-Authored-By: Claude Opus 5.5 <noreply@anthropic.com>
Claude-Session: https://claude.ai/code/session_01CHDvF8BfHwPLkrFs9S3ECm
Parts:
- D10, D11: symbol AVO:BAT54C_D -> AVO:BAT54C_D_1aa644
- J1: symbol AVO:USB-C_J -> AVO:USB-C_J_cb921f
- J2: symbol AVO:BATERÍA_J -> AVO:BATERÍA_J_ac1e8e
- K1: symbol AVO:G6KU-2F-Y_K -> AVO:G6KU-2F-Y_K_ae8a75
- Q1, Q2: symbol AVO:AO3401A_Q -> AVO:AO3401A_Q_71681c
- Q10, Q14, Q17, Q3: symbol AVO:AO3401A_Q -> AVO:AO3401A_Q_bcf332
- Q11, Q13: symbol AVO:AO3400A_Q -> AVO:AO3400A_Q_71681c
- Q12, Q15, Q16, Q18: symbol AVO:2N7002_Q -> AVO:2N7002_Q_71681c
- U1: symbol AVO:BQ51013BRHLR_U -> AVO:BQ51013BRHLR_U_606a23
- U2: symbol AVO:BQ24072RGTR_U -> AVO:BQ24072RGTR_U_4b171e
- U3: symbol AVO:RT9080-33GJ5_U -> AVO:RT9080-33GJ5_U_7ca22f
- U4: symbol AVO:ESP32-C6-MINI-1U-N4_U -> AVO:ESP32-C6-MINI-1U-N4_U_91bf48
- U5: symbol AVO:BNO085_U -> AVO:BNO085_U_cee500
- U6: symbol AVO:USBLC6-2SC6_U -> AVO:USBLC6-2SC6_U_7dacad
Connections:
- net AD_SRC: now also Q1.2 (S), Q2.2 (S); no longer Q1.3 (D), Q2.3 (D)
- net VBUS: now also Q1.3 (D); no longer Q1.2 (S)
- net VIN5: now also Q2.3 (D); no longer Q2.2 (S)
Changed lines of the file:
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@@
 	)
 	(symbol
-		(lib_id "AVO:BAT54C_D")
+		(lib_id "AVO:BAT54C_D_1aa644")
 		(at 43.18 275.59 0)
 		(unit 1)
@@
 	)
 	(symbol
-		(lib_id "AVO:BAT54C_D")
+		(lib_id "AVO:BAT54C_D_1aa644")
 		(at 91.44 275.59 0)
 		(unit 1)
@@
 	)
 	(symbol
-		(lib_id "AVO:G6KU-2F-Y_K")
+		(lib_id "AVO:G6KU-2F-Y_K_ae8a75")
 		(at 142.24 280.67 0)
 		(unit 1)
@@
 	)
 	(symbol
-		(lib_id "AVO:AO3401A_Q")
+		(lib_id "AVO:AO3401A_Q_bcf332")
 		(at 194.31 275.59 0)
 		(unit 1)
@@
 	)
 	(symbol
-		(lib_id "AVO:AO3400A_Q")
+		(lib_id "AVO:AO3400A_Q_71681c")
 		(at 241.3 275.59 0)
 		(unit 1)
@@
 	)
 	(symbol
-		(lib_id "AVO:2N7002_Q")
+		(lib_id "AVO:2N7002_Q_71681c")
 		(at 43.18 299.72 0)
 		(unit 1)
@@
 	)
 	(symbol
-		(lib_id "AVO:AO3400A_Q")
+		(lib_id "AVO:AO3400A_Q_71681c")
 		(at 91.44 299.72 0)
 		(unit 1)
@@
 	)
 	(symbol
-		(lib_id "AVO:AO3401A_Q")
+		(lib_id "AVO:AO3401A_Q_bcf332")
 		(at 137.16 299.72 0)
 		(unit 1)
@@
 	)
 	(symbol
-		(lib_id "AVO:2N7002_Q")
+		(lib_id "AVO:2N7002_Q_71681c")
 		(at 184.15 299.72 0)
 		(unit 1)
@@
 	)
 	(symbol
-		(lib_id "AVO:AO3401A_Q")
+		(lib_id "AVO:AO3401A_Q_bcf332")
 		(at 231.14 299.72 0)
 		(unit 1)
@@
 	)
 	(symbol
-		(lib_id "AVO:2N7002_Q")
+		(lib_id "AVO:2N7002_Q_71681c")
 		(at 43.18 313.69 0)
 		(unit 1)
@@
 	)
 	(symbol
-		(lib_id "AVO:USB-C_J")
+		(lib_id "AVO:USB-C_J_cb921f")
 		(at 307.34 49.53 0)
 		(unit 1)
@@
 	)
 	(symbol
-		(lib_id "AVO:AO3401A_Q")
+		(lib_id "AVO:AO3401A_Q_71681c")
 		(at 355.6 36.83 0)
 		(unit 1)
@@
 	)
 	(symbol
-		(lib_id "AVO:AO3401A_Q")
+		(lib_id "AVO:AO3401A_Q_71681c")
 		(at 403.86 36.83 0)
 		(unit 1)
@@
 	)
 	(symbol
-		(lib_id "AVO:USBLC6-2SC6_U")
+		(lib_id "AVO:USBLC6-2SC6_U_7dacad")
 		(at 453.39 39.37 0)
 		(unit 1)
@@
 	)
 	(symbol
-		(lib_id "AVO:BATERÍA_J")
+		(lib_id "AVO:BATERÍA_J_ac1e8e")
 		(at 43.18 177.8 0)
 		(unit 1)
@@
 	)
 	(symbol
-		(lib_id "AVO:2N7002_Q")
+		(lib_id "AVO:2N7002_Q_71681c")
 		(at 88.9 177.8 0)
 		(unit 1)
@@
 	)
 	(symbol
-		(lib_id "AVO:RT9080-33GJ5_U")
+		(lib_id "AVO:RT9080-33GJ5_U_7ca22f")
 		(at 132.08 179.07 0)
 		(unit 1)
@@
 	)
 	(symbol
-		(lib_id "AVO:AO3401A_Q")
+		(lib_id "AVO:AO3401A_Q_bcf332")
 		(at 304.8 139.7 0)
 		(unit 1)
@@
 	)
 	(symbol
-		(lib_id "AVO:BNO085_U")
+		(lib_id "AVO:BNO085_U_cee500")
 		(at 360.68 157.48 0)
 		(unit 1)
@@
 	)
 	(symbol
-		(lib_id "AVO:BQ51013BRHLR_U")
+		(lib_id "AVO:BQ51013BRHLR_U_606a23")
 		(at 49.53 49.53 0)
 		(unit 1)
@@
 	)
 	(symbol
-		(lib_id "AVO:BQ24072RGTR_U")
+		(lib_id "AVO:BQ24072RGTR_U_4b171e")
 		(at 565.15 45.72 0)
 		(unit 1)
@@
 	)
 	(symbol
-		(lib_id "AVO:ESP32-C6-MINI-1U-N4_U")
+		(lib_id "AVO:ESP32-C6-MINI-1U-N4_U_91bf48")
 		(at 576.58 172.72 0)
 		(unit 1)

Commit message: PCB cincha REV B: ESP32-C3-MINI-1U-N4, LSM6DS3TR-C + MMC5983MA por I²C, corte de batería con MOSFET; REV A (C6) congelada
- REV A copiada tal cual a hardware/girth/PCB_REV_A_C6 (puerta superada en e9e5166).
- U4 ESP32-C3-MINI-1U-N4 (C2911374, 1191 uds. en JLCPCB el 2026-10-29); nueva asignación de GPIO.
- IMU: BNO085 (19,50 US$, 80 uds.) sustituido por LSM6DS3TR-C + MMC5983MA (I²C), mismos datos de 9 ejes.
- Relé biestable sustituido por enclavamiento PMOS/NMOS (reed por flanco, 5 V de carga, PWR_HOLD).
- R6/R7 a 3k3 (piezas Basic). Ficheros de fabricación con nombres C3.

Co-Authored-By: Claude Opus 5.5 <noreply@anthropic.com>
Claude-Session: https://claude.ai/code/session_01CHDvF8BfHwPLkrFs9S3ECm
Parts:
- removed C32, C43: 100n, AVO:C_0402_1005Metric, symbol AVO:C_avo
- removed K1: G6KU-2F-Y DC3, AVO:Relay_DPDT_Omron_G6K-2F-Y, symbol AVO:G6KU-2F-Y_K_ae8a75
- removed Q12, Q15, Q18: 2N7002, AVO:SOT-23, symbol AVO:2N7002_Q_71681c
- removed Q13: AO3400A, AVO:SOT-23, symbol AVO:AO3400A_Q_71681c
- removed Q14, Q17, Q3: AO3401A, AVO:SOT-23, symbol AVO:AO3401A_Q_bcf332
- removed R14, R22, R23, R24, R25, R26, R27, R44, R45: 10k, AVO:R_0402_1005Metric, symbol AVO:R_avo
- removed R28, R29: 4k7, AVO:R_0402_1005Metric, symbol AVO:R_avo
- removed R30, R46, R47, R48, R53, R54: 100k, AVO:R_0402_1005Metric, symbol AVO:R_avo
- removed R51: 1M, AVO:R_0402_1005Metric, symbol AVO:R_avo
- removed R52: 10R, AVO:R_0805_2012Metric, symbol AVO:R_avo
- removed R55: 1k, AVO:R_0402_1005Metric, symbol AVO:R_avo
- removed Y1: 32,768 kHz 12,5 pF, AVO:Crystal_SMD_3215-2Pin_3.2x1.5mm, symbol AVO:Crystal_avo
- added R42: 1M, AVO:R_0402_1005Metric, symbol AVO:R_avo
- added R43: 100k, AVO:R_0402_1005Metric, symbol AVO:R_avo
- added U7: MMC5983MA, AVO:MEMSIC_MMC5983MA_LGA-16_3x3mm_P0.5mm, symbol AVO:MMC5983MA_U_48c675
- C27, C28: value 22p -> 100n; LCSC C1555 -> C1525
- C29: value 100n -> 1u; LCSC C1525 -> C52923
- C30: value 100n -> 10u 6V3; footprint AVO:C_0402_1005Metric -> AVO:C_0603_1608Metric; LCSC C1525 -> C19702
- C31: value 4u7 -> 100n; footprint AVO:C_0603_1608Metric -> AVO:C_0402_1005Metric; LCSC C19666 -> C1525
- C40: value 220u 6V3 polímero -> 10u 6V3; footprint AVO:CP_EIA-3528-21_Kemet-B -> AVO:C_0603_1608Metric; LCSC C79111 -> C19702
- C41: value 220u 6V3 polímero -> 2u2; footprint AVO:CP_EIA-3528-21_Kemet-B -> AVO:C_0603_1608Metric; LCSC C79111 -> C23630
- D1: value LED verde -> LED rojo; MPN (none) -> KT-0603R
- D10, D11: value BAT54C -> BAV70; symbol AVO:BAT54C_D_1aa644 -> AVO:BAV70_D_1aa644; LCSC C2135 -> C68978
- R20, R21: value 10k -> 4k7; LCSC C25744 -> C25900
- R40: value 0R -> 1M; footprint AVO:R_0805_2012Metric -> AVO:R_0402_1005Metric; LCSC C17477 -> C26083
- R41: value 0R -> 1M; footprint AVO:R_0805_2012Metric -> AVO:R_0402_1005Metric; LCSC C17477 -> C26083; now fitted
- R6: value 3k6 -> 3k3; LCSC C25891 -> C25890
- R7: value 3k4 -> 3k3; LCSC C4940 -> C25890
- U4: value ESP32-C6-MINI-1U-N4 -> ESP32-C3-MINI-1U-N4; footprint AVO:ESP32-C6-MINI-1U -> AVO:ESP32-C3-MINI-1U; symbol AVO:ESP32-C6-MINI-1U-N4_U_91bf48 -> AVO:ESP32-C3-MINI-1U-N4_U_f334d7; LCSC C7558096 -> C2911374; MPN ESP32-C6-MINI-1U-N4 (alt. -H4 C20627095) -> ESP32-C3-MINI-1U-N4 (alt. ESP32-C3-MINI-1U-H4 C3013922)
- U5: value BNO085 -> LSM6DS3TR-C; footprint AVO:CEVA_BNO08x_LGA-28_5.2x3.8mm_P0.5mm -> AVO:LGA-14_3x2.5mm_P0.5mm_LayoutBorder3x4y; symbol AVO:BNO085_U_cee500 -> AVO:LSM6DS3TR-C_U_b4fcf8; LCSC C5189642 -> C967633; MPN BNO085 (alt. BNO086) -> LSM6DS3TR-C (alt. LSM6DSV16XTR C5267406)
Connections:
- net GPIO8 is gone; now on net LED: R13.1, U4.22 (IO8 LED)
- net RLY_NC is gone; now on net REED_PULSE: R41.1
- net RLY_NO is gone; now on net BAT_RAW: R40.1
- net RLY_ON_D is gone; now on net REED_PULSE: D11.1 (A1)
- net SS_G is gone; now on net PWR_PG: Q10.1 (G)
- net +3V3: now also C27.1, C28.1, C29.1, C31.1, D1.2 (A), R20.2, R21.2, U5.12 (CS), U5.5 (VDDIO), U5.8 (VDD), U7.13 (VDDIO), U7.2 (VDD), U7.4 (SPI_CS)
- net BAT_ADC: now also U4.6 (IO3 BAT_ADC); no longer U4.5 (IO2 BAT_ADC)
- net BAT_RAW: now also Q10.2 (S)
- net CHG_PG: now also U4.18 (IO4 CHG_PG); no longer U4.6 (IO3 CHG_PG)
- net CHG_STAT: now also U4.5 (IO2 CHG_STAT); no longer U4.9 (IO4 CHG_STAT)
- net GND: now also C41.2, R41.2, U5.1 (SDO/SA0), U5.3 (SCx), U5.6 (GND), U5.7 (GND), R42.2, R43.2, U7.11 (GND), U7.9 (GND); no longer D1.1 (K), U5.10 (CLKSEL0), U5.25 (GND)
- net IMU_INT: now also U5.4 (INT1); no longer U5.14 (H_INTN)
- net LED: no longer U4.20 (IO15 LED)
- net QI_CHG: now also U4.16 (IO10 QI_CHG); no longer U4.28 (IO22 QI_CHG)
- net REED: now also U4.13 (IO1 REED); no longer U4.15 (IO6 REED)
- net REED_HI: now also C40.1; no longer D10.1 (A1)
- net USB_DM: now also U4.26 (IO18 D-); no longer U4.17 (IO12 D-)
- net USB_DP: now also U4.27 (IO19 D+); no longer U4.18 (IO13 D+)
- net VIN5: now also D10.1 (A1); no longer D10.2 (A2)
- net I2C_SCL: now reaches U4.21 (IO7 SCL)
- net I2C_SCL: now also R21.1, U5.13 (SCL), U7.1 (SCL)
- net REED_PULSE: now reaches D11.2 (A2)
- net REED_PULSE: now also C40.2
- removed net BAT_SW: Q10.2 (S), R40.2, R41.2
- net IMU_BOOTN renamed I2C_SDA
- net I2C_SDA: now also U4.20 (IO6 SDA), U5.14 (SDA), U7.16 (SDA); no longer U5.4 (BOOTN)
- net IMU_CAP: no longer names the net of U5.9 (INT2)
- net IMU_CS: no longer names the net of U4.24 (NC)
- net IMU_CS: no longer U5.18 (H_CSN)
- removed net IMU_ENV_SCL: U5.15 (ENV_SCL)
- removed net IMU_ENV_SDA: U5.16 (ENV_SDA)
- removed net IMU_MISO: U4.27 (IO21 MISO), U5.20 (MISO/SDA)
- removed net IMU_MOSI: U4.26 (IO20 MOSI), U5.17 (MOSI/SA0)
- removed net IMU_PS1: R21.1, U5.5 (PS1)
- net IMU_PWR_N: no longer names the net of U4.10 (NC)
- net IMU_RST: no longer names the net of U5.11 (SDO_Aux)
- net IMU_RST: no longer U4.13 (IO1 IMU_RST)
- net IMU_SCK: no longer names the net of U4.25 (NC)
- net IMU_SCK: no longer U5.19 (SCK/SCL)
- removed net IMU_VDD: C29.1, C30.1, C31.1, R20.2, R21.2, U5.28 (VDDIO), U5.3 (VDD)
- removed net IMU_WAKE: U4.16 (IO7 IMU_WAKE), U5.6 (PS0/WAKE)
- removed net IMU_XIN: C27.1, U5.27 (XIN32)
- removed net IMU_XOUT: C28.1, U5.26 (XOUT32)
- removed net K_A: C40.2, C41.2
- net K_B renamed PWR_PG
- net PWR_PG: now also R40.2
- net LED_A renamed LED_K
- net LED_K: now also D1.1 (K); no longer D1.2 (A)
- net RLY_GB renamed PWR_G
- net PWR_G: now also C41.1, D10.3 (K), R42.1
- net RLY_OFF: no longer names the net of U4.29 (NC)
- net RLY_ON renamed PWR_HOLD
- net PWR_HOLD: now also D10.2 (A2), R43.1
- removed net RLY_P: C40.1, C41.1, D10.3 (K)
- new net MAG_CAP: C30.1, U7.10 (CAP)
- no-connect marks 21 -> 29
Other:
- note added: "CORTE DE BATERÍA: enclavamiento con MOSFET (reed · 5 V · PWR_HOLD)"
- note added: "ESP32-C3-MINI-1U-N4 · arranque · LED · pruebas"
- note added: "IMU LSM6DS3TR-C + MMC5983MA (I²C)"
- note removed: "CORTE DE BATERÍA: relé biestable G6KU"
- note removed: "ESP32-C6-MINI-1U · arranque · LED · pruebas"
- note removed: "IMU BNO085 (SPI) · alimentación conmutada"
- title: AVO GIRTH · placa de la cincha · REV A -> AVO GIRTH · placa de la cincha · REV B
- moved on the sheet: C23, C24, C25, C27, C28, C29, C30, C31, C40, C41, D1, D10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

Commit message: PCB cincha REV B: huella LGA-14L propia (0,25 mm entre pads; la genérica dejaba 0,1 mm); zip del firmware sin la carpeta build
Co-Authored-By: Claude Opus 5.5 <noreply@anthropic.com>
Claude-Session: https://claude.ai/code/session_01CHDvF8BfHwPLkrFs9S3ECm
Parts:
- U5: footprint AVO:LGA-14_3x2.5mm_P0.5mm_LayoutBorder3x4y -> AVO:ST_LGA-14L_2.5x3mm_P0.5mm
Changed lines of the file:
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@@
 		(property
 			"Footprint"
-			"AVO:LGA-14_3x2.5mm_P0.5mm_LayoutBorder3x4y"
+			"AVO:ST_LGA-14L_2.5x3mm_P0.5mm"
 			(at 304.8 147.32 0)
 			(hide yes)

Commit message: Cincha REV B: SCL en GPIO2 (la hoja del ESP32-C3-MINI-1 pide GPIO2 = 1 al arrancar; el pull-up I²C lo garantiza), CHG_STAT en GPIO7
Co-Authored-By: Claude Opus 5.5 <noreply@anthropic.com>
Claude-Session: https://claude.ai/code/session_01CHDvF8BfHwPLkrFs9S3ECm
Parts:
- U4: symbol AVO:ESP32-C3-MINI-1U-N4_U_f334d7 -> AVO:ESP32-C3-MINI-1U-N4_U_668a8a
Connections:
- net CHG_STAT: now also U4.21 (IO7 CHG_STAT); no longer U4.5 (IO2 CHG_STAT)
- net I2C_SCL: now also U4.5 (IO2 SCL); no longer U4.21 (IO7 SCL)
Changed lines of the file:
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@@
 	)
 	(symbol
-		(lib_id "AVO:ESP32-C3-MINI-1U-N4_U_f334d7")
+		(lib_id "AVO:ESP32-C3-MINI-1U-N4_U_668a8a")
 		(at 574.04 166.37 0)
 		(unit 1)
@@
 	)
 	(global_label
-		"CHG_STAT"
+		"I2C_SCL"
 		(shape passive)
 		(at 553.72 143.51 180)
@@
 	)
 	(global_label
-		"I2C_SCL"
+		"CHG_STAT"
 		(shape passive)
 		(at 553.72 156.21 180)
