File: hardware/girth/PCB/kicad/AVO_GIRTH_PCB.kicad_sch (KiCad schematic)
At the start: 94 parts, among them J1 USB-C 16P, J2 BATERÍA 1S, Q1 AO3401A, Q10 AO3401A, Q11 AO3400A, Q16 2N7002, Q2 AO3401A, SW1 REED (1), SW2 REED (2), U1 BQ51013BRHLR, U2 BQ24072RGTR, U3 RT9080-33GJ5, U4 ESP32-C3-MINI-1U-N4, U5 LSM6DS3TR-C, U6 USBLC6-2SC6, U7 MMC5983MA

Commit message: Cincha REV B: red del reed revisada (D12 aísla la lectura, R44 limita la corriente, R45/D13 rearman en ~2 s, C40/C41 10× menores) y firmware: no despertar por reed ya cerrado, IMU al ritmo del dato listo, magnetómetro opcional
Corrige los fallos de una revisión independiente: con el reed cerrado la placa no se podía apagar (despertar por
nivel) y tras sacar la cápsula el reed no la volvía a encender durante 10–25 s.

Co-Authored-By: Claude Opus 5.5 <noreply@anthropic.com>
Claude-Session: https://claude.ai/code/session_01CHDvF8BfHwPLkrFs9S3ECm
Parts:
- added D12, D13: BAV70, AVO:SOT-23, symbol AVO:BAV70_D_1aa644
- added R44: 220R, AVO:R_0402_1005Metric, symbol AVO:R_avo
- added R45: 1M, AVO:R_0402_1005Metric, symbol AVO:R_avo
- C40: value 10u 6V3 -> 2u2; LCSC C19702 -> C23630
- C41: value 2u2 -> 220n; footprint AVO:C_0603_1608Metric -> AVO:C_0402_1005Metric; LCSC C23630 -> C16772
- R41, R42: value 1M -> 10M; LCSC C26083 -> C26082
Connections:
- net GND: now also D13.1 (A1), D13.2 (A2), R45.2
- net REED_HI: now also D12.1 (A1), D12.2 (A2); no longer C40.1
- net REED_PULSE: now also D13.3 (K)
- new net REED_C: D12.3 (K), R44.1, R45.1
- new net REED_CR: C40.1, R44.2
Other:
- moved on the sheet: C40, C41, Q10, Q11, R40, R41, R42, R43
