File: hardware/girth/PCB/kicad/AVO_GIRTH_PCB.kicad_pcb (KiCad board)
At the start: 4 copper layers, 65.5 x 43.5 mm, 122 parts, among them J1 USB-C 16P, J2 BATERÍA 1S, K1 G6KU-2F-Y DC3, Q1 AO3401A, Q10 AO3401A, Q11 AO3400A, Q12 2N7002, Q13 AO3400A, Q14 AO3401A, Q15 2N7002, Q16 2N7002, Q17 AO3401A, Q18 2N7002, Q2 AO3401A, Q3 AO3401A, SW1 REED (1), SW2 REED (2), U1 BQ51013BRHLR, U2 BQ24072RGTR, U3 RT9080-33GJ5, U4 ESP32-C6-MINI-1U-N4, U5 BNO085, U6 USBLC6-2SC6, Y1 32,768 kHz 12,5 pF

Commit message: PCB cincha: resultados de KiCad 9 de f1d04a0 (puerta: false) [skip ci]
Parts:
- removed C32, C43: 100n, AVO:C_0402_1005Metric
- removed K1: G6KU-2F-Y DC3, AVO:Relay_DPDT_Omron_G6K-2F-Y
- removed Q12, Q15, Q18: 2N7002, AVO:SOT-23
- removed Q13: AO3400A, AVO:SOT-23
- removed Q14, Q17, Q3: AO3401A, AVO:SOT-23
- removed R14, R22, R23, R24, R25, R26, R27, R44, R45: 10k, AVO:R_0402_1005Metric
- removed R28, R29: 4k7, AVO:R_0402_1005Metric
- removed R30, R46, R47, R48, R53, R54: 100k, AVO:R_0402_1005Metric
- removed R51: 1M, AVO:R_0402_1005Metric
- removed R52: 10R, AVO:R_0805_2012Metric
- removed R55: 1k, AVO:R_0402_1005Metric
- removed Y1: 32,768 kHz 12,5 pF, AVO:Crystal_SMD_3215-2Pin_3.2x1.5mm
- added R42: 1M, AVO:R_0402_1005Metric, F.Cu at (86.8, 85.8)
- added R43: 100k, AVO:R_0402_1005Metric, F.Cu at (87.4, 82.4)
- added U7: MMC5983MA, AVO:MEMSIC_MMC5983MA_LGA-16_3x3mm_P0.5mm, F.Cu at (95.0, 90.4)
- C27, C28: value 22p -> 100n
- C29: value 100n -> 1u
- C30: value 100n -> 10u 6V3; footprint AVO:C_0402_1005Metric -> AVO:C_0603_1608Metric
- C31: value 4u7 -> 100n; footprint AVO:C_0603_1608Metric -> AVO:C_0402_1005Metric
- C40: value 220u 6V3 polímero -> 10u 6V3; footprint AVO:CP_EIA-3528-21_Kemet-B -> AVO:C_0603_1608Metric
- C41: value 220u 6V3 polímero -> 2u2; footprint AVO:CP_EIA-3528-21_Kemet-B -> AVO:C_0603_1608Metric
- D1: value LED verde -> LED rojo
- D10, D11: value BAT54C -> BAV70
- R20, R21: value 10k -> 4k7
- R40, R41: value 0R -> 1M; footprint AVO:R_0805_2012Metric -> AVO:R_0402_1005Metric
- R6: value 3k6 -> 3k3
- R7: value 3k4 -> 3k3
- U4: value ESP32-C6-MINI-1U-N4 -> ESP32-C3-MINI-1U-N4; footprint AVO:ESP32-C6-MINI-1U -> AVO:ESP32-C3-MINI-1U
- U5: value BNO085 -> LSM6DS3TR-C; footprint AVO:CEVA_BNO08x_LGA-28_5.2x3.8mm_P0.5mm -> AVO:LGA-14_3x2.5mm_P0.5mm_LayoutBorder3x4y
- moved D10 26.4 mm to (87.8, 89.0)
- moved Q11 25.6 mm to (84.4, 89.0)
- moved C40 15.6 mm to (92.4, 85.4)
- moved R40 14.6 mm to (81.0, 86.2), turned to 0 degrees
- moved C41 11.0 mm to (84.4, 85.8), turned to 0 degrees
- moved R41 10.5 mm to (92.4, 82.8), turned to 0 degrees
- moved R21 9.70 mm to (105.1, 99.0), turned to 90 degrees
- moved R20 8.66 mm to (104.0, 99.0), turned to 90 degrees
- moved D11 7.47 mm to (89.4, 85.4)
- moved C31 7.33 mm to (95.0, 88.0), turned to 0 degrees
- moved C29 7.08 mm to (92.6, 90.4), turned to 90 degrees
- moved C27 4.51 mm to (97.4, 97.0)
- moved C28 4.46 mm to (102.6, 97.0)
- moved U4 2.00 mm to (113.6, 107.0)
- moved C30 1.34 mm to (95.0, 93.0)
Connections:
- C27 pad 1: IMU_XIN -> +3V3
- C28 pad 1: IMU_XOUT -> +3V3
- C29 pad 1: IMU_VDD -> +3V3
- C30 pad 1: IMU_VDD -> MAG_CAP
- C31 pad 1: IMU_VDD -> +3V3
- C40 pad 1: RLY_P -> REED_HI
- C40 pad 2: K_A -> REED_PULSE
- C41 pad 1: RLY_P -> PWR_G
- C41 pad 2: K_A -> GND
- D1 pad 1: GND -> LED_K
- D1 pad 2: LED_A -> +3V3
- D10 pad 1: REED_HI -> VIN5
- D10 pad 2: VIN5 -> PWR_HOLD
- D10 pad 3: RLY_P -> PWR_G
- D11 pad 1: RLY_ON_D -> REED_PULSE
- D11 pad 2: unconnected-(D11-A2-Pad2) -> REED_PULSE
- D11 pad 3: RLY_GB -> PWR_G
- Q10 pad 1: SS_G -> PWR_PG
- Q10 pad 2: BAT_SW -> BAT_RAW
- Q11 pad 1: RLY_GB -> PWR_G
- Q11 pad 3: K_B -> PWR_PG
- R13 pad 1: GPIO8 -> LED
- R15 pad 2: LED_A -> LED_K
- R20 pad 1: IMU_BOOTN -> I2C_SDA
- R20 pad 2: IMU_VDD -> +3V3
- R21 pad 1: IMU_PS1 -> I2C_SCL
- R21 pad 2: IMU_VDD -> +3V3
- R40 pad 1: RLY_NO -> BAT_RAW
- R40 pad 2: BAT_SW -> PWR_PG
- R41 pad 1: RLY_NC -> REED_PULSE
- R41 pad 2: BAT_SW -> GND
- U4 pad 10: IMU_PWR_N -> unconnected-(U4-NC-Pad10)
- U4 pad 13: IMU_RST -> REED
- U4 pad 15: REED -> unconnected-(U4-NC-Pad15)
- U4 pad 16: IMU_WAKE -> QI_CHG
- U4 pad 17: USB_DM -> unconnected-(U4-NC-Pad17)
- U4 pad 18: USB_DP -> CHG_PG
- U4 pad 19: RLY_ON -> PWR_HOLD
- U4 pad 20: LED -> I2C_SDA
- U4 pad 21: unconnected-(U4-NC-Pad21) -> I2C_SCL
- U4 pad 22: GPIO8 -> LED
- U4 pad 24: IMU_CS -> unconnected-(U4-NC-Pad24)
- U4 pad 25: IMU_SCK -> unconnected-(U4-NC-Pad25)
- U4 pad 26: IMU_MOSI -> USB_DM
- U4 pad 27: IMU_MISO -> USB_DP
- U4 pad 28: QI_CHG -> unconnected-(U4-NC-Pad28)
- U4 pad 29: RLY_OFF -> unconnected-(U4-NC-Pad29)
- U4 pad 5: BAT_ADC -> CHG_STAT
- U4 pad 6: CHG_PG -> BAT_ADC
- U4 pad 9: CHG_STAT -> unconnected-(U4-NC-Pad9)
- U5 pad 1: unconnected-(U5-NC-Pad1) -> GND
- U5 pad 10: GND -> unconnected-(U5-OCS_Aux-Pad10)
- U5 pad 11: IMU_RST -> unconnected-(U5-SDO_Aux-Pad11)
- U5 pad 12: unconnected-(U5-NC-Pad12) -> +3V3
- U5 pad 13: unconnected-(U5-NC-Pad13) -> I2C_SCL
- U5 pad 14: IMU_INT -> I2C_SDA
- U5 pad 3: IMU_VDD -> GND
- U5 pad 4: IMU_BOOTN -> IMU_INT
- U5 pad 5: IMU_PS1 -> +3V3
- U5 pad 6: IMU_WAKE -> GND
- U5 pad 7: unconnected-(U5-NC-Pad7) -> GND
- U5 pad 8: unconnected-(U5-NC-Pad8) -> +3V3
- U5 pad 9: IMU_CAP -> unconnected-(U5-INT2-Pad9)
Routing:
- net RLY_OFF: track 56.7 -> 0.00 mm, vias 5 -> 0
- net PWR_HOLD: track 0.00 -> 52.5 mm, vias 0 -> 3
- net K_A: track 50.4 -> 0.00 mm, vias 4 -> 0
- net K_B: track 45.3 -> 0.00 mm, vias 3 -> 0
- net RLY_GB: track 45.3 -> 0.00 mm, vias 3 -> 0
- net IMU_VDD: track 41.5 -> 0.00 mm, vias 3 -> 0
- net RLY_ON: track 39.7 -> 0.00 mm, vias 2 -> 0
- net I2C_SDA: track 0.00 -> 39.4 mm, vias 0 -> 2
- net IMU_SCK: track 39.2 -> 0.00 mm, vias 3 -> 0
- net RLY_P: track 37.8 -> 0.00 mm, vias 2 -> 0
- net IMU_PWR_N: track 34.4 -> 0.00 mm, vias 3 -> 0
- net I2C_SCL: track 0.00 -> 33.4 mm, vias 0 -> 3
- net IMU_WAKE: track 31.3 -> 0.00 mm, vias 2 -> 0
- net IMU_RST: track 28.7 -> 0.00 mm, vias 3 -> 0
- net BAT_SW: track 27.3 -> 0.00 mm
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Other:
- board text added: "AVO GIRTH · REV B · ESP32-C3 · 2026-10-29"
- board text removed: "AVO GIRTH · REV A · 2026-10-29"

Commit message: PCB cincha: resultados de KiCad 9 de 968fe80 (puerta: false) [skip ci]
Parts:
- U5: footprint AVO:LGA-14_3x2.5mm_P0.5mm_LayoutBorder3x4y -> AVO:ST_LGA-14L_2.5x3mm_P0.5mm
Routing:
- net +3V3: track 112.1 -> 123.3 mm
- net REED_HI: track 48.2 -> 42.0 mm
- net I2C_SDA: track 39.4 -> 35.1 mm, vias 2 -> 3
- net BAT_RAW: track 44.1 -> 47.7 mm
- net REED: track 26.5 -> 29.6 mm
- net I2C_SCL: track 33.4 -> 35.2 mm
- net PWR_HOLD: track 52.5 -> 54.2 mm
- net GND: track 45.1 -> 43.5 mm
- net EN: track 18.9 -> 18.2 mm, vias 2 -> 0

Commit message: PCB cincha: resultados de KiCad 9 de 01f8093 (puerta: false) [skip ci]
Connections:
- U4 pad 21: I2C_SCL -> CHG_STAT
- U4 pad 5: CHG_STAT -> I2C_SCL
Routing:
- net I2C_SCL: track 35.2 -> 44.2 mm, vias 3 -> 4
- net BOOT: track 26.6 -> 33.8 mm
- net IMU_INT: track 39.9 -> 34.8 mm
- net GND: track 43.5 -> 48.5 mm
- net CHG_STAT: track 29.6 -> 34.1 mm
- net PWR_HOLD: track 54.2 -> 51.6 mm
- net +3V3: track 123.3 -> 121.5 mm
- net REED: track 29.6 -> 28.6 mm
- net U0TX: track 18.8 -> 19.6 mm
- net BAT_ADC: track 13.8 -> 13.2 mm

Commit message: PCB cincha: resultados de KiCad 9 de 6b01cb8 (puerta: true) [skip ci]
Routing:
- net QI_ADEN: track 7.20 -> 12.6 mm
- net QI_AC1: track 14.1 -> 17.2 mm
- net QI_ILIM: track 0.00 -> 2.99 mm, vias 0 -> 2
- net QI_CHG: vias 2 -> 4

Commit message: PCB cincha: resultados de KiCad 9 de ffe91b8 (puerta: false) [skip ci]
Parts:
- added D12: BAV70, AVO:SOT-23, F.Cu at (85.0, 93.0)
- added D13: BAV70, AVO:SOT-23, F.Cu at (90.0, 93.0)
- added R44: 220R, AVO:R_0402_1005Metric, F.Cu at (82.4, 92.4)
- added R45: 1M, AVO:R_0402_1005Metric, F.Cu at (87.4, 92.4)
- C40: value 10u 6V3 -> 2u2
- C41: value 2u2 -> 220n; footprint AVO:C_0603_1608Metric -> AVO:C_0402_1005Metric
- R41, R42: value 1M -> 10M
Connections:
- C40 pad 1: REED_HI -> REED_CR
Routing:
- net IMU_INT: track 34.8 -> 0.00 mm, vias 2 -> 0
- net REED_CR: track 0.00 -> 15.5 mm, vias 0 -> 2
- net REED_PULSE: track 10.8 -> 18.7 mm
- net REED_C: track 0.00 -> 6.38 mm, vias 0 -> 2
- net QI_ADEN: track 12.6 -> 6.25 mm
- net +3V3: track 121.5 -> 117.7 mm
- net PWR_G: track 15.9 -> 12.8 mm, vias 2 -> 0
- net QI_ILIM: track 2.99 -> 0.00 mm, vias 2 -> 0
- net I2C_SCL: track 44.2 -> 41.7 mm, vias 4 -> 3
- net CHG_STAT: track 34.1 -> 32.1 mm
- net REED_HI: track 42.4 -> 40.7 mm
- net QI_AC1: track 17.2 -> 18.2 mm
- net BOOT: track 33.8 -> 34.6 mm
- net PWR_HOLD: track 51.6 -> 52.3 mm
- net EN: track 18.4 -> 17.7 mm
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
Commit message: PCB cincha: resultados de KiCad 9 de 227d414 (puerta: true) [skip ci]
Routing:
- net IMU_INT: track 0.00 -> 25.8 mm, vias 0 -> 2
- net +3V3: track 117.7 -> 124.0 mm, vias 6 -> 8
- net QI_ADEN: track 6.25 -> 11.5 mm
- net QI_CHG: track 40.0 -> 43.4 mm, vias 2 -> 6
- net QI_ILIM: track 0.00 -> 2.91 mm, vias 0 -> 2
- net CHG_PG: track 33.0 -> 35.0 mm, vias 3 -> 6
- net VBUS: track 69.0 -> 70.9 mm, vias 7 -> 9
- net U0RX: track 19.3 -> 17.5 mm
- net GND: track 48.0 -> 46.4 mm
- net REED: track 28.7 -> 28.4 mm, vias 2 -> 3
