File: hardware/girth/PCB/kicad/AVO_GIRTH_PCB_ruteado.kicad_pcb (KiCad board)
At the start: 4 copper layers, 65.5 x 43.5 mm, 98 parts, among them J1 USB-C 16P, J2 BATERÍA 1S, Q1 AO3401A, Q10 AO3401A, Q11 AO3400A, Q16 2N7002, Q2 AO3401A, SW1 REED (1), SW2 REED (2), U1 BQ51013BRHLR, U2 BQ24072RGTR, U3 RT9080-33GJ5, U4 ESP32-C3-MINI-1U-N4, U5 LSM6DS3TR-C, U6 USBLC6-2SC6, U7 MMC5983MA

Commit message: Cincha: quitado el resto del tramo colgante de QI_CHG; los flujos del CI reintentan el guardado si chocan en la rama (la compilación de ffe91b8 fue correcta pero no se guardó)
Co-Authored-By: Claude Opus 5.5 <noreply@anthropic.com>
Claude-Session: https://claude.ai/code/session_01CHDvF8BfHwPLkrFs9S3ECm
Routing:
- net QI_CHG: track 43.3 -> 42.6 mm
Changed lines of the file:
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@@
-	)
-	(segment
-		(start 119.2 108.6)
-		(end 118.5483 108.6)
-		(width 0.2)
-		(layer "F.Cu")
-		(net 34)
 	)
 	(segment
