File: hardware/girth/PCB/AUDITORIA_REV_B/resultados_ci/rev_b1/AVO_GIRTH_PCB_REV_B1_zonas_rellenas.kicad_pcb (KiCad board)
At the start: 4 copper layers, 65.5 x 43.5 mm, 98 parts, among them J1 USB-C 16P, J2 BATERÍA 1S, Q1 AO3401A, Q10 AO3401A, Q11 AO3400A, Q16 2N7002, Q2 AO3401A, SW1 REED (1), SW2 REED (2), U1 BQ51013BRHLR, U2 BQ24072RGTR, U3 RT9080-33GJ5, U4 ESP32-C3-MINI-1U-N4, U5 LSM6DS3TR-C, U6 USBLC6-2SC6, U7 MMC5983MA

Commit message: Auditoría REV B: evidencias del CI de 7be067a [skip ci]
Parts:
- C41: value 220n -> 470n
- R40: value 1M -> 100k
Changed lines of the file:
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@@
 			)
 		)
-		(property "Value" "220n"
+		(property "Value" "470n"
 			(at 0 1.06 0)
 			(layer "F.Fab")
@@
 			)
 		)
-		(property "LCSC" "C16772"
-			(at 0 0 0)
-			(layer "F.Fab")
-			(hide yes)
-			(effects
-				(font
-					(size 0.6 0.6)
-					(thickness 0.1)
-				)
-			)
-		)
-		(property "MPN" "220n"
+		(property "LCSC" "C1543"
+			(at 0 0 0)
+			(layer "F.Fab")
+			(hide yes)
+			(effects
+				(font
+					(size 0.6 0.6)
+					(thickness 0.1)
+				)
+			)
+		)
+		(property "MPN" "470n"
 			(at 0 0 0)
 			(layer "F.Fab")
@@
 			)
 		)
-		(property "Value" "1M"
+		(property "Value" "100k"
 			(at 0 1.07 0)
 			(layer "F.Fab")
@@
 			)
 		)
-		(property "LCSC" "C26083"
-			(at 0 0 0)
-			(layer "F.Fab")
-			(hide yes)
-			(effects
-				(font
-					(size 0.6 0.6)
-					(thickness 0.1)
-				)
-			)
-		)
-		(property "MPN" "1M"
-			(at 0 0 0)
-			(layer "F.Fab")
+		(property "LCSC" "C25741"
+			(at 0 0 0)
+			(layer "F.Fab")
+			(hide yes)
+			(effects
+				(font
+					(size 0.6 0.6)
+					(thickness 0.1)
+				)
+			)
+		)
+		(property "MPN" "100k"
+			(at 0 0 0)
+			(layer "F.Fab")
