File: hardware/girth/PCB/AUDITORIA_REV_B/corregida/kicad/AVO_GIRTH_PCB.kicad_pcb (KiCad board)
At the start: 4 copper layers, 65.5 x 43.5 mm, 98 parts, among them J1 USB-C 16P, J2 BATERÍA 1S, Q1 AO3401A, Q10 AO3401A, Q11 AO3400A, Q16 2N7002, Q2 AO3401A, SW1 REED (1), SW2 REED (2), U1 BQ51013BRHLR, U2 BQ24072RGTR, U3 RT9080-33GJ5, U4 ESP32-C3-MINI-1U-N4, U5 LSM6DS3TR-C, U6 USBLC6-2SC6, U7 MMC5983MA

Commit message: Auditoría REV B: REV B.1 con C41 = 470 nF y R40 = 100 k (simulado: 0/200 caídas en reinicios), BOM de la B.1 con el algoritmo de jlc.py, SPICE y existencias de la B.1 en el CI, pico de encendido en los resultados, README ≤ 2 µA
Co-Authored-By: Claude Opus 5.5 <noreply@anthropic.com>
Claude-Session: https://claude.ai/code/session_01CHDvF8BfHwPLkrFs9S3ECm
Parts:
- C41: value 220n -> 470n
- R40: value 1M -> 100k
Changed lines of the file:
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@@
 		(property
 			"Value"
-			"1M"
+			"100k"
 			(at 0 1.07 0)
 			(layer "F.Fab")
@@
 		(property
 			"LCSC"
-			"C26083"
+			"C25741"
 			(at 0 0 0)
 			(layer "F.Fab")
@@
 		(property
 			"MPN"
-			"1M"
+			"100k"
 			(at 0 0 0)
 			(layer "F.Fab")
@@
 		(property
 			"Value"
-			"220n"
+			"470n"
 			(at 0 1.06 0)
 			(layer "F.Fab")
@@
 		(property
 			"LCSC"
-			"C16772"
+			"C1543"
 			(at 0 0 0)
 			(layer "F.Fab")
@@
 		(property
 			"MPN"
-			"220n"
-			(at 0 0 0)
-			(layer "F.Fab")
+			"470n"
+			(at 0 0 0)
+			(layer "F.Fab")
