File: hardware/girth/PCB/AUDITORIA_REV_B/corregida/kicad/AVO_GIRTH_PCB.kicad_sch (KiCad schematic)
At the start: 98 parts, among them J1 USB-C 16P, J2 BATERÍA 1S, Q1 AO3401A, Q10 AO3401A, Q11 AO3400A, Q16 2N7002, Q2 AO3401A, SW1 REED (1), SW2 REED (2), U1 BQ51013BRHLR, U2 BQ24072RGTR, U3 RT9080-33GJ5, U4 ESP32-C3-MINI-1U-N4, U5 LSM6DS3TR-C, U6 USBLC6-2SC6, U7 MMC5983MA

Commit message: Auditoría REV B: REV B.1 con C41 = 470 nF y R40 = 100 k (simulado: 0/200 caídas en reinicios), BOM de la B.1 con el algoritmo de jlc.py, SPICE y existencias de la B.1 en el CI, pico de encendido en los resultados, README ≤ 2 µA
Co-Authored-By: Claude Opus 5.5 <noreply@anthropic.com>
Claude-Session: https://claude.ai/code/session_01CHDvF8BfHwPLkrFs9S3ECm
Parts:
- C41: value 220n -> 470n; LCSC C16772 -> C1543
- R40: value 1M -> 100k; LCSC C26083 -> C25741
Changed lines of the file:
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@@
 		(dnp no)
 		(property "Reference" "C41" (at 356.87 257.81 0) (effects (font (size 1.27 1.27)) (justify left)))
-		(property "Value" "220n" (at 356.87 260.35 0) (effects (font (size 1 1)) (justify left)))
+		(property "Value" "470n" (at 356.87 260.35 0) (effects (font (size 1 1)) (justify left)))
 		(property
 			"Footprint"
@@
 		(property "Datasheet" "" (at 354.33 259.08 0) (hide yes) (effects (font (size 1.27 1.27))))
 		(property "Description" "" (at 354.33 259.08 0) (hide yes) (effects (font (size 1.27 1.27))))
-		(property "LCSC" "C16772" (at 354.33 259.08 0) (hide yes) (effects (font (size 1.27 1.27))))
+		(property "LCSC" "C1543" (at 354.33 259.08 0) (hide yes) (effects (font (size 1.27 1.27))))
 		(property "MPN" "" (at 354.33 259.08 0) (hide yes) (effects (font (size 1.27 1.27))))
 		(pin "1")
@@
 		(dnp no)
 		(property "Reference" "R40" (at 381 260.35 0) (effects (font (size 1.27 1.27)) (justify left)))
-		(property "Value" "1M" (at 381 262.89 0) (effects (font (size 1 1)) (justify left)))
+		(property "Value" "100k" (at 381 262.89 0) (effects (font (size 1 1)) (justify left)))
 		(property
 			"Footprint"
@@
 		(property "Datasheet" "" (at 378.46 261.62 0) (hide yes) (effects (font (size 1.27 1.27))))
 		(property "Description" "" (at 378.46 261.62 0) (hide yes) (effects (font (size 1.27 1.27))))
-		(property "LCSC" "C26083" (at 378.46 261.62 0) (hide yes) (effects (font (size 1.27 1.27))))
+		(property "LCSC" "C25741" (at 378.46 261.62 0) (hide yes) (effects (font (size 1.27 1.27))))
 		(property "MPN" "" (at 378.46 261.62 0) (hide yes) (effects (font (size 1.27 1.27))))
 		(pin "1")

Commit message: Auditoría REV B: C41 de la REV B.1 = C47339 (CL05A474KP5NNNC 470 nF 0402); C1543 resultó ser 820 pF (comprobado en el CI)
Co-Authored-By: Claude Opus 5.5 <noreply@anthropic.com>
Claude-Session: https://claude.ai/code/session_01CHDvF8BfHwPLkrFs9S3ECm
Parts:
- C41: LCSC C1543 -> C47339
Changed lines of the file:
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@@
 		(property "Datasheet" "" (at 354.33 259.08 0) (hide yes) (effects (font (size 1.27 1.27))))
 		(property "Description" "" (at 354.33 259.08 0) (hide yes) (effects (font (size 1.27 1.27))))
-		(property "LCSC" "C1543" (at 354.33 259.08 0) (hide yes) (effects (font (size 1.27 1.27))))
+		(property "LCSC" "C47339" (at 354.33 259.08 0) (hide yes) (effects (font (size 1.27 1.27))))
 		(property "MPN" "" (at 354.33 259.08 0) (hide yes) (effects (font (size 1.27 1.27))))
 		(pin "1")
