File: hardware/back/V4/PCB/kicad/AVO_BACK_V4_PCB.kicad_sch (KiCad schematic)
At the start: 99 parts, among them J1 USB-C 16P, J2 BATERÍA 1S, J3 microSD DM3AT, J4 URTK1.2 (8 hilos), Q1 AO3401A, Q2 AO3401A, Q3 AO3401A, Q4 AO3401A, U1 BQ51013BRHLR, U2 BQ24072RGTR, U3 TLV75733PDBVR, U4 ESP32-S3-MINI-1U-N8, U6 USBLC6-2SC6, U7 RT9080-33GJ5, U8 DRV5032FADBZR

Commit message: AVO BACK V4 PCB REV B: sin Qi ni Hall; 3 contactos en el fondo (SYS y BAT en la cola, GND aparte) con TVS; REV A congelada en PCB_REV_A_QI
Soporte del chaleco = puente SYS–BAT (encendido); base de carga = cargador externo entre BAT y GND. USB-C del taller con
el BQ24072. Colocación nueva sin bloque Qi.

Co-Authored-By: Claude Opus 5.5 <noreply@anthropic.com>
Claude-Session: https://claude.ai/code/session_01CHDvF5XNd4qsah8Nejvp3z
Parts:
- removed C1, C2: 100n C0G 50V, AVO:C_1206_3216Metric, symbol AVO:C_avo
- removed C10, C7: 470n 25V, AVO:C_0603_1608Metric, symbol AVO:C_avo
- removed C11, C8: 22n 50V, AVO:C_0402_1005Metric, symbol AVO:C_avo
- removed C12, C13, C15: 10u 25V, AVO:C_0603_1608Metric, symbol AVO:C_avo
- removed C14, C16, C33: 100n, AVO:C_0402_1005Metric, symbol AVO:C_avo
- removed C17: 1u, AVO:C_0402_1005Metric, symbol AVO:C_avo
- removed C3: 47n C0G 50V, AVO:C_1206_3216Metric, symbol AVO:C_avo
- removed C4: 2n2 C0G 50V, AVO:C_0805_2012Metric, symbol AVO:C_avo
- removed C5: 1n C0G 50V, AVO:C_0603_1608Metric, symbol AVO:C_avo
- removed C6, C9: 10n 50V, AVO:C_0402_1005Metric, symbol AVO:C_avo
- removed L1: BOBINA Qi (1), AVO:WirePad_D1.5_Drill0.8, symbol AVO:Pad_avo
- removed L2: BOBINA Qi (2), AVO:WirePad_D1.5_Drill0.8, symbol AVO:Pad_avo
- removed Q1, Q2: AO3401A, AVO:SOT-23, symbol AVO:AO3401A_Q_71681c
- removed R1: 330R, AVO:R_0402_1005Metric, symbol AVO:R_avo
- removed R2: 200R, AVO:R_0402_1005Metric, symbol AVO:R_avo
- removed R3: 20k, AVO:R_0402_1005Metric, symbol AVO:R_avo
- removed R4: 100k, AVO:R_0402_1005Metric, symbol AVO:R_avo
- removed RT1: NTC 10k B3380, AVO:R_0402_1005Metric, symbol AVO:R_avo
- removed U1: BQ51013BRHLR, AVO:Texas_VQFN-RHL-20_ThermalVias, symbol AVO:BQ51013BRHLR_U_606a23
- removed U8: DRV5032FADBZR, AVO:SOT-23, symbol AVO:DRV5032FADBZR_U_225eda
- added D2, D3: TVS 5 V, AVO:D_SOD-323, symbol AVO:TVS_D_bafa22
- added P1: CONTACTO SYS, AVO:AVO_Contacto_M2_Tornillo, symbol AVO:Pad_avo
- added P2: CONTACTO BAT, AVO:AVO_Contacto_M2_Tornillo, symbol AVO:Pad_avo
- added P3: CONTACTO GND, AVO:AVO_Contacto_M2_Tornillo, symbol AVO:Pad_avo
- U4: symbol AVO:ESP32-S3-MINI-1U-N8_U_edcc57 -> AVO:ESP32-S3-MINI-1U-N8_U_f0d859
Connections:
- net VIN5 is gone; now on net VBUS: C18.1, U2.13 (IN)
- net BAT_F: now also D3.1 (K), P2.1; no longer Q3.3 (D)
- net GND: now also D2.2 (A), D3.2 (A), P3.1
- net HALL: no longer names the net of U4.5 (IO1)
- net QI_CHG: no longer names the net of U4.36 (IO40)
- new net SYS_IN: D2.1 (K), P1.1, Q3.3 (D)
- no-connect marks 17 -> 19
Other:
- note added: "BATERÍA: PTC hacia el contacto BAT · protección de polaridad del contacto SYS · medida por ADC"
- note added: "CARGADOR CON CAMINO DE POTENCIA (BQ24072) · solo USB-C del taller · batería 1S 2000 mAh (654060)"
- note added: "CONTACTOS DEL FONDO (REV B): SYS y BAT en la cola, GND aparte · chaleco = puente SYS–BAT · base de carga = cargador entre BAT y GND"
- note added: "USB-C (taller: programación, datos y carga) · ESD"
- note removed: "BATERÍA: PTC + protección de polaridad · medida por ADC"
- note removed: "CARGADOR CON CAMINO DE POTENCIA (BQ24072) · batería 1S 2000 mAh (654060)"
- note removed: "RECEPTOR Qi (BQ51013B) · bobina 30 × 23 bajo la placa · USB por AD/AD-EN"
- note removed: "SENSOR DE SOPORTE: Hall DRV5032FA (imanes del soporte)"
- note removed: "USB-C (programación y carga) · ESD"
- title: AVO BACK V4 · placa de la espalda · REV A -> AVO BACK V4 · placa de la espalda · REV B
- moved on the sheet: C21, C22, C24, C25, C26, C27, C28, C34, C40, C41, C60, C61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
